Commit message: added hardware interface

File: robots/panda_arm_hand.urdf.xacro (robot description, xacro)
@@ -9,5 +9,5 @@
   <xacro:if value="$(arg load_gripper)">
     <xacro:include filename="$(find franka_panda_description)/robots/hand.xacro"/>
-    <xacro:hand ns="panda" rpy="0 0 ${-pi/4}" connected_to="panda_link8"/>
+    <xacro:hand ns="$(arg robot_name)" rpy="0 0 ${-pi/4}" connected_to="$(arg robot_name)_link8"/>
   </xacro:if>
   <xacro:if value="$(arg load_gazebo)">
@@ -19,5 +19,5 @@
   </xacro:if>
   <xacro:unless value="$(arg load_gazebo)">
-    <xacro:panda_arm />
+    <xacro:panda_arm arm_id="$(arg robot_name)" />
   </xacro:unless>
 </robot>

File: ros2_control/franka_panda_torque.ros2_control.xacro (robot description, xacro)
@@ -16,5 +16,5 @@
         </hardware>
       </xacro:unless>
-      <joint name="panda_joint1">
+      <joint name="${prefix}_joint1">
         <command_interface name="effort">
           <param name="min">-87</param>
@@ -23,5 +23,5 @@
         <state_interface name="position"/>
       </joint>
-      <joint name="panda_joint2">
+      <joint name="${prefix}_joint2">
         <command_interface name="effort">
           <param name="min">-87</param>
@@ -30,5 +30,5 @@
         <state_interface name="position"/>
       </joint>
-      <joint name="panda_joint3">
+      <joint name="${prefix}_joint3">
         <command_interface name="effort">
           <param name="min">-87</param>
@@ -37,5 +37,5 @@
         <state_interface name="position"/>
       </joint>
-      <joint name="panda_joint4">
+      <joint name="${prefix}_joint4">
         <command_interface name="effort">
           <param name="min">-87</param>
@@ -44,5 +44,5 @@
         <state_interface name="position"/>
       </joint>
-      <joint name="panda_joint5">
+      <joint name="${prefix}_joint5">
         <command_interface name="effort">
           <param name="min">-12</param>
@@ -51,5 +51,5 @@
         <state_interface name="position"/>
       </joint>
-      <joint name="panda_joint6">
+      <joint name="${prefix}_joint6">
         <command_interface name="effort">
           <param name="min">-12</param>
@@ -58,5 +58,5 @@
         <state_interface name="position"/>
       </joint>
-      <joint name="panda_joint7">
+      <joint name="${prefix}_joint7">
         <command_interface name="effort">
           <param name="min">-12</param>
@@ -66,5 +66,5 @@
       </joint>
       <xacro:if value="$(arg use_gripper)">
-	<joint name="panda_finger_joint1">
+	<joint name="${prefix}_finger_joint1">
           <command_interface name="effort">
             <param name="min">-20</param>
@@ -73,5 +73,5 @@
           <state_interface name="position"/>
 	</joint>
-	<joint name="panda_finger_joint2">
+	<joint name="${prefix}_finger_joint2">
           <command_interface name="effort">
             <param name="min">-20</param>
