Commit message: perform collision checking only for hand and fingers

File: robots/panda_arm.xacro (robot description, xacro)
@@ -26,5 +26,5 @@
       <collision>
         <geometry>
-          <mesh filename="package://${description_pkg}/meshes/collision/link0.stl"/>
+          <!-- <mesh filename="package://${description_pkg}/meshes/collision/link0.stl"/> -->
         </geometry>
       </collision>
@@ -45,5 +45,5 @@
       <collision>
         <geometry>
-          <mesh filename="package://${description_pkg}/meshes/collision/link1.stl"/>
+          <!-- <mesh filename="package://${description_pkg}/meshes/collision/link1.stl"/> -->
         </geometry>
       </collision>
@@ -71,5 +71,5 @@
       <collision>
         <geometry>
-          <mesh filename="package://${description_pkg}/meshes/collision/link2.stl"/>
+          <!-- <mesh filename="package://${description_pkg}/meshes/collision/link2.stl"/> -->
         </geometry>
       </collision>
@@ -97,5 +97,5 @@
       <collision>
         <geometry>
-          <mesh filename="package://${description_pkg}/meshes/collision/link3.stl"/>
+          <!-- <mesh filename="package://${description_pkg}/meshes/collision/link3.stl"/> -->
         </geometry>
       </collision>
@@ -123,5 +123,5 @@
       <collision>
         <geometry>
-          <mesh filename="package://${description_pkg}/meshes/collision/link4.stl"/>
+          <!-- <mesh filename="package://${description_pkg}/meshes/collision/link4.stl"/> -->
         </geometry>
       </collision>
@@ -149,5 +149,5 @@
       <collision>
         <geometry>
-          <mesh filename="package://${description_pkg}/meshes/collision/link5.stl"/>
+          <!-- <mesh filename="package://${description_pkg}/meshes/collision/link5.stl"/> -->
         </geometry>
       </collision>
@@ -175,5 +175,5 @@
       <collision>
         <geometry>
-          <mesh filename="package://${description_pkg}/meshes/collision/link6.stl"/>
+          <!-- <mesh filename="package://${description_pkg}/meshes/collision/link6.stl"/> -->
         </geometry>
       </collision>
@@ -201,5 +201,5 @@
       <collision>
         <geometry>
-          <mesh filename="package://${description_pkg}/meshes/collision/link7.stl"/>
+          <!-- <mesh filename="package://${description_pkg}/meshes/collision/link7.stl"/> -->
         </geometry>
       </collision>

Commit message: eliminate errors during loading

File: robots/panda_arm.xacro (robot description, xacro)
@@ -24,9 +24,11 @@
         </geometry>
       </visual>
-      <collision>
-        <geometry>
-          <!-- <mesh filename="package://${description_pkg}/meshes/collision/link0.stl"/> -->
-        </geometry>
-      </collision>
+      <!--
+      <collision>
+        <geometry>
+          <mesh filename="package://${description_pkg}/meshes/collision/link0.stl"/>
+        </geometry>
+      </collision>
+      -->
       <xacro:unless value="${in_gazebo == 'false'}">
         <inertial>
@@ -43,9 +45,11 @@
         </geometry>
       </visual>
-      <collision>
-        <geometry>
-          <!-- <mesh filename="package://${description_pkg}/meshes/collision/link1.stl"/> -->
-        </geometry>
-      </collision>
+      <!--
+      <collision>
+        <geometry>
+          <mesh filename="package://${description_pkg}/meshes/collision/link1.stl"/>
+        </geometry>
+      </collision>
+      -->
       <inertial>
         <origin xyz="3.875e-03 2.081e-03 -0.1750" rpy="0 0 0"/>
@@ -69,9 +73,11 @@
         </geometry>
       </visual>
-      <collision>
-        <geometry>
-          <!-- <mesh filename="package://${description_pkg}/meshes/collision/link2.stl"/> -->
-        </geometry>
-      </collision>
+      <!--
+      <collision>
+        <geometry>
+          <mesh filename="package://${description_pkg}/meshes/collision/link2.stl"/>
+        </geometry>
+      </collision>
+      -->
       <inertial>
         <origin xyz="-3.141e-03 -2.872e-02 3.495e-03" rpy="0 0 0"/>
@@ -95,9 +101,11 @@
         </geometry>
       </visual>
-      <collision>
-        <geometry>
-          <!-- <mesh filename="package://${description_pkg}/meshes/collision/link3.stl"/> -->
-        </geometry>
-      </collision>
+      <!--
+      <collision>
+        <geometry>
+          <mesh filename="package://${description_pkg}/meshes/collision/link3.stl"/>
+        </geometry>
+      </collision>
+      -->
       <inertial>
         <origin xyz="2.7518e-02 3.9252e-02 -6.6502e-02" rpy="0 0 0"/>
@@ -121,9 +129,11 @@
         </geometry>
       </visual>
-      <collision>
-        <geometry>
-          <!-- <mesh filename="package://${description_pkg}/meshes/collision/link4.stl"/> -->
-        </geometry>
-      </collision>
+      <!--
+      <collision>
+        <geometry>
+          <mesh filename="package://${description_pkg}/meshes/collision/link4.stl"/>
+        </geometry>
+      </collision>
+      -->
       <inertial>
         <origin xyz="-5.317e-02 1.04419e-01 2.7454e-02" rpy="0 0 0"/>
@@ -147,9 +157,11 @@
         </geometry>
       </visual>
-      <collision>
-        <geometry>
-          <!-- <mesh filename="package://${description_pkg}/meshes/collision/link5.stl"/> -->
-        </geometry>
-      </collision>
+      <!--
+      <collision>
+        <geometry>
+          <mesh filename="package://${description_pkg}/meshes/collision/link5.stl"/>
+        </geometry>
+      </collision>
+      -->
       <inertial>
         <origin xyz="-1.1953e-02 4.1065e-02 -3.8437e-02" rpy="0 0 0"/>
@@ -173,9 +185,11 @@
         </geometry>
       </visual>
-      <collision>
-        <geometry>
-          <!-- <mesh filename="package://${description_pkg}/meshes/collision/link6.stl"/> -->
-        </geometry>
-      </collision>
+      <!--
+      <collision>
+        <geometry>
+          <mesh filename="package://${description_pkg}/meshes/collision/link6.stl"/>
+        </geometry>
+      </collision>
+      -->
       <inertial>
         <origin xyz="6.0149e-02 -1.4117e-02 -1.0517e-02" rpy="0 0 0"/>
@@ -199,9 +213,11 @@
         </geometry>
       </visual>
-      <collision>
-        <geometry>
-          <!-- <mesh filename="package://${description_pkg}/meshes/collision/link7.stl"/> -->
-        </geometry>
-      </collision>
+      <!--
+      <collision>
+        <geometry>
+          <mesh filename="package://${description_pkg}/meshes/collision/link7.stl"/>
+        </geometry>
+      </collision>
+      -->
       <inertial>
         <origin xyz="1.0517e-02 -4.252e-03 6.1597e-02" rpy="0 0 0"/>
