Commit message: remove damping and friction because mujoco uses them

File: robots/hand.xacro (robot description, xacro)
@@ -68,5 +68,5 @@
       <axis xyz="0 1 0"/>
       <limit effort="20" lower="0.0" upper="0.04" velocity="0.2"/>
-      <dynamics damping="500.0" friction="0.0"/>
+      <dynamics damping="0.0" friction="0.0"/>
     </joint>
     <joint name="${ns}_finger_joint2" type="prismatic">
@@ -76,5 +76,5 @@
       <axis xyz="0 -1 0"/>
       <limit effort="20" lower="0.0" upper="0.04" velocity="0.2"/>
-      <dynamics damping="500.0" friction="0.0"/>
+      <dynamics damping="0.0" friction="0.0"/>
       <mimic joint="${ns}_finger_joint1" />
     </joint>

File: robots/panda_arm.xacro (robot description, xacro)
@@ -65,5 +65,5 @@
       <axis xyz="0 0 1"/>
       <limit effort="87" lower="-2.8973" upper="2.8973" velocity="2.1750"/>
-      <dynamics damping="10.0" friction="5.0"/>
+      <dynamics damping="0.0" friction="0.0"/>
     </joint>
     <link name="${arm_id}_link2">
@@ -93,5 +93,5 @@
       <axis xyz="0 0 1"/>
       <limit effort="87" lower="-1.7628" upper="1.7628" velocity="2.1750"/>
-      <dynamics damping="5.0" friction="2.0"/>
+      <dynamics damping="0.0" friction="0.0"/>
     </joint>
     <link name="${arm_id}_link3">
@@ -121,5 +121,5 @@
       <axis xyz="0 0 1"/>
       <limit effort="87" lower="-2.8973" upper="2.8973" velocity="2.1750"/>
-      <dynamics damping="5.0" friction="2.0"/>
+      <dynamics damping="0.0" friction="0.0"/>
     </joint>
     <link name="${arm_id}_link4">
@@ -149,5 +149,5 @@
       <axis xyz="0 0 1"/>
       <limit effort="87" lower="-3.0718" upper="-0.0698" velocity="2.1750"/>
-      <dynamics damping="1.0" friction="0.5"/>
+      <dynamics damping="0.0" friction="0.0"/>
     </joint>
     <link name="${arm_id}_link5">
@@ -177,5 +177,5 @@
       <axis xyz="0 0 1"/>
       <limit effort="12" lower="-2.8973" upper="2.8973" velocity="2.6100"/>
-      <dynamics damping="2.0" friction="1.0"/>
+      <dynamics damping="0.0" friction="0.0"/>
     </joint>
     <link name="${arm_id}_link6">
@@ -205,5 +205,5 @@
       <axis xyz="0 0 1"/>
       <limit effort="12" lower="-0.0175" upper="3.7525" velocity="2.6100"/>
-      <dynamics damping="1.0" friction="0.5"/>
+      <dynamics damping="0.0" friction="0.0"/>
     </joint>
     <link name="${arm_id}_link7">
@@ -233,5 +233,5 @@
       <axis xyz="0 0 1"/>
       <limit effort="12" lower="-2.8973" upper="2.8973" velocity="2.6100"/>
-      <dynamics damping="1.0" friction="0.5"/>
+      <dynamics damping="0.0" friction="0.0"/>
     </joint>
     <link name="${arm_id}_link8">
